File: jar-of-fireflies.brd (EAGLE design)
At the start: 50 x 50 mm, 21 parts, among them U1 ATTINY45

Commit message: Rev 1.1: fixed swapped 1M and 1K resistors, incremented version number.
Parts:
- R4: value 1K -> 1M
- R5: value 1M -> 1K
- R6: value 1k -> 1K
Other:
- board text added: "Jar of Fireflies V1.1 https://git.io/fireflies"
- board text removed: "Jar of Fireflies V1.0 https://git.io/fireflies"
Changed lines of the file:
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@@
 <wire x1="3.60555" y1="50" x2="0" y2="46.39445" width="0" layer="20" curve="90"/>
 <circle x="25" y="25" radius="28" width="0.254" layer="21"/>
-<text x="25" y="19.5" size="2.25" layer="51" font="vector" align="center">Jar of Fireflies V1.0
+<text x="25" y="19.5" size="2.25" layer="51" font="vector" align="center">Jar of Fireflies V1.1
 https://git.io/fireflies</text>
 <text x="25" y="17.6" size="2" layer="30" font="vector" rot="MR0" align="center">joefitz@securinghardware.com
@@
 <attribute name="VALUE" x="15.856" y="8.871" size="0.8128" layer="21" font="vector" ratio="15" rot="R180"/>
 </element>
-<element name="R4" library="SparkFun-Passives" package="AXIAL-0.4" value="1K" x="36.43" y="8.49" smashed="yes">
+<element name="R4" library="SparkFun-Passives" package="AXIAL-0.4" value="1M" x="36.43" y="8.49" smashed="yes">
 <attribute name="NAME" x="35.795" y="8.109" size="0.8128" layer="25" font="vector" ratio="15" align="bottom-right"/>
 <attribute name="VALUE" x="38.716" y="8.109" size="0.8128" layer="21" font="vector" ratio="15" align="bottom-right"/>
 </element>
-<element name="R5" library="SparkFun-Passives" package="AXIAL-0.4" value="1M" x="36.43" y="11.03" smashed="yes">
+<element name="R5" library="SparkFun-Passives" package="AXIAL-0.4" value="1K" x="36.43" y="11.03" smashed="yes">
 <attribute name="NAME" x="35.795" y="10.649" size="0.8128" layer="25" font="vector" ratio="15" align="bottom-right"/>
 <attribute name="VALUE" x="38.716" y="10.649" size="0.8128" layer="21" font="vector" ratio="15" align="bottom-right"/>
 </element>
-<element name="R6" library="SparkFun-Passives" package="AXIAL-0.4" value="1k" x="36.43" y="5.95" smashed="yes" rot="R180">
+<element name="R6" library="SparkFun-Passives" package="AXIAL-0.4" value="1K" x="36.43" y="5.95" smashed="yes" rot="R180">
 <attribute name="NAME" x="35.795" y="6.331" size="0.8128" layer="25" font="vector" ratio="15" rot="R180"/>
 <attribute name="VALUE" x="38.716" y="6.331" size="0.8128" layer="21" font="vector" ratio="15" rot="R180"/>

Commit message: up to rev 1.2. Gave up on touch sense, replaced with through-hole switch, fewer components!
Parts:
- removed R4: 1M, SparkFun-Passives:AXIAL-0.4
- removed R5, R6: 1K, SparkFun-Passives:AXIAL-0.4
- S1: value SWITCH-MOMENTARY-2SMD-1101NE -> SWITCH-MOMENTARY-2PTH; device SparkFun-Electromechanical:TACTILE-SWITCH-1101NE -> SparkFun-Electromechanical:TACTILE-PTH
- moved S1 3.57 mm to (36.0, 10.8), turned to 0 degrees
Connections:
- removed net N$11: R6.P$2, S1.2, U1.1
- removed net N$5: R5.P$1, U1.3
- removed net RING: R4.P$2, R5.P$2
- net N$4: now also S1.3; no longer R4.P$1
- net VCC: no longer R6.P$1
Routing:
- net N$11: track 11.7 -> 0.00 mm
- net RING: track 7.48 -> 0.00 mm, vias 1 -> 0
- net N$5: track 2.54 -> 0.00 mm
- net N$4: track 2.54 -> 4.04 mm
Other:
- board text added: "Jar of Fireflies V1.2 https://git.io/fireflies"
- board text removed: "Jar of Fireflies V1.1 https://git.io/fireflies"
Changed lines of the file:
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@@
 <wire x1="3.60555" y1="50" x2="0" y2="46.39445" width="0" layer="20" curve="90"/>
 <circle x="25" y="25" radius="28" width="0.254" layer="21"/>
-<text x="25" y="19.5" size="2.25" layer="51" font="vector" align="center">Jar of Fireflies V1.1
+<text x="25" y="19.5" size="2.25" layer="51" font="vector" align="center">Jar of Fireflies V1.2
 https://git.io/fireflies</text>
 <text x="25" y="17.6" size="2" layer="30" font="vector" rot="MR0" align="center">joefitz@securinghardware.com
@@
 <attribute name="VALUE" x="15.856" y="8.871" size="0.8128" layer="21" font="vector" ratio="15" rot="R180"/>
 </element>
-<element name="R4" library="SparkFun-Passives" package="AXIAL-0.4" value="1M" x="36.43" y="8.49" smashed="yes">
-<attribute name="NAME" x="35.795" y="8.109" size="0.8128" layer="25" font="vector" ratio="15" align="bottom-right"/>
-<attribute name="VALUE" x="38.716" y="8.109" size="0.8128" layer="21" font="vector" ratio="15" align="bottom-right"/>
-</element>
-<element name="R5" library="SparkFun-Passives" package="AXIAL-0.4" value="1K" x="36.43" y="11.03" smashed="yes">
-<attribute name="NAME" x="35.795" y="10.649" size="0.8128" layer="25" font="vector" ratio="15" align="bottom-right"/>
-<attribute name="VALUE" x="38.716" y="10.649" size="0.8128" layer="21" font="vector" ratio="15" align="bottom-right"/>
-</element>
-<element name="R6" library="SparkFun-Passives" package="AXIAL-0.4" value="1K" x="36.43" y="5.95" smashed="yes" rot="R180">
-<attribute name="NAME" x="35.795" y="6.331" size="0.8128" layer="25" font="vector" ratio="15" rot="R180"/>
-<attribute name="VALUE" x="38.716" y="6.331" size="0.8128" layer="21" font="vector" ratio="15" rot="R180"/>
-</element>
-<element name="S1" library="SparkFun-Electromechanical" package="TACTILE-SWITCH-1101NE" value="SWITCH-MOMENTARY-2SMD-1101NE" x="36.4" y="14.35" smashed="yes" rot="R180">
-<attribute name="PROD_ID" value="SWCH-00815" x="36.4" y="14.35" size="1.778" layer="27" rot="R180" display="off"/>
+<element name="S1" library="SparkFun-Electromechanical" package="TACTILE-PTH" value="SWITCH-MOMENTARY-2PTH" x="36.05" y="10.8" smashed="yes">
+<attribute name="PROD_ID" value=" SWCH-08441" x="36.05" y="10.8" size="1.778" layer="27" display="off"/>
 </element>
 <element name="U1" library="SparkFun-DigitalIC" package="DIP08" value="ATTINY45" x="25" y="9.76" smashed="yes" rot="R90">
@@
 <contactref element="R3" pad="P$1"/>
 <wire x1="21.19" y1="8.49" x2="18.65" y2="8.49" width="0.4064" layer="1"/>
-</signal>
-<signal name="N$4">
-<contactref element="U1" pad="2"/>
-<contactref element="R4" pad="P$1"/>
-<wire x1="31.35" y1="8.49" x2="28.81" y2="8.49" width="0.4064" layer="1"/>
-</signal>
-<signal name="N$5">
-<contactref element="U1" pad="3"/>
-<contactref element="R5" pad="P$1"/>
-<wire x1="31.35" y1="11.03" x2="28.81" y2="11.03" width="0.4064" layer="1"/>
 </signal>
 <signal name="N$6">
@@
 <signal name="VCC">
 <contactref element="U1" pad="8"/>
-<contactref element="R6" pad="P$1"/>
 <contactref element="BAT1" pad="1"/>
 <polygon width="0.4064" layer="16">
@@
 <contactref element="U1" pad="4"/>
 <contactref element="BAT1" pad="2"/>
-<contactref element="S1" pad="1"/>
 <polygon width="0.4064" layer="1">
 <vertex x="0" y="0"/>
@@
 <via x="3" y="10" extent="1-16" drill="1"/>
 <via x="40" y="3" extent="1-16" drill="1"/>
-</signal>
-<signal name="N$11">
-<contactref element="U1" pad="1"/>
-<contactref element="R6" pad="P$2"/>
-<contactref element="R6" pad="P$2"/>
-<wire x1="31.35" y1="5.95" x2="28.81" y2="5.95" width="0.4064" layer="1"/>
-<contactref element="S1" pad="2"/>
-<wire x1="31.35" y1="5.95" x2="33.25" y2="7.85" width="0.4064" layer="1" curve="90"/>
-<wire x1="33.25" y1="7.85" x2="33.25" y2="14.35" width="0.4064" layer="1"/>
-</signal>
-<signal name="RING">
-<contactref element="R4" pad="P$2"/>
-<contactref element="R5" pad="P$2"/>
-<wire x1="41.51" y1="11.03" x2="41.51" y2="8.49" width="0.4064" layer="1"/>
-<via x="45" y="5" extent="1-16" drill="3.2"/>
-<wire x1="41.51" y1="8.49" x2="45" y2="5" width="0.4064" layer="1"/>
+<contactref element="S1" pad="1"/>
 </signal>
 <signal name="N$8">
@@
 <via x="45" y="45" extent="1-16" drill="3.2"/>
 </signal>
+<signal name="N$4">
+<contactref element="U1" pad="2"/>
+<contactref element="S1" pad="3"/>
+<wire x1="28.81" y1="8.49" x2="32.7988" y2="8.49" width="0.4064" layer="16"/>
+<wire x1="32.7988" y1="8.49" x2="32.7988" y2="8.5394" width="0.4064" layer="16"/>
+</signal>
 </signals>
